Commit message: rebase commits
updated focal length


Odometry + joint state publisher

added robot model


renaming do->update

File: ROS_ws/src/sPrinter_description/urdf/sPrinter.xacro (robot description, xacro)
@@ -414,3 +414,24 @@
     <child link="lens_focal_static_frame"/>
   </joint>
+  <!--middle frame joint-->
+  <joint name="lens_frame_middle_joint" type="fixed">
+    <origin xyz="-0.2535  0.0 0.0" rpy="0 0 0"/>
+    <parent link="lens_Xrot_frame_1"/>
+    <child link="lens_frame_middle"/>
+  </joint>
+  <!--focal work frame joint-->
+  <joint name="lens_focal_work_frame_joint" type="fixed">
+    <origin rpy="0 0 0" xyz="0.0 0.0 -0.50" />
+            <!-- z: ohniskova vzdialenost -->
+    <parent link="lens_frame_middle"/>
+    <child link="lens_focal_work_frame"/>
+  </joint>
+  <!--focal static frame joint-->
+  <joint name="lens_focal_static_frame_joint" type="fixed">
+    <origin rpy="0 0 0" xyz="0.753764 0.0 0.05" />
+            <!-- z: 55cm - ohniskova vzdialenost = 5cm nad zemou-->
+            <!-- x: 0.753764 je pri 0.615m vysunuti sosovky v x (HOME) ... pod lens_midle frame-->
+    <parent link="base_link"/>
+    <child link="lens_focal_static_frame"/>
+  </joint>
 </robot>

Commit message: diff drive controller is working Other controllers need to be fixed so robot doesnt tilt back

File: ROS_ws/src/sPrinter_description/urdf/sPrinter.xacro (robot description, xacro)
@@ -285,26 +285,4 @@
     </collision>
   </link>
-  <!--  frame in the middle of the lens-->
-  <link name="lens_frame_middle">
-    <inertial>
-      <origin xyz="0.0 0.0 0.0" rpy="0 0 0"/>
-      <mass value="0.0"/>
-      <inertia ixx="0.0" iyy="0.0" izz="0.0" ixy="0.0" iyz="0.0" ixz="0.0"/>
-    </inertial>
-  </link>
-  <link name="lens_focal_work_frame">
-    <inertial>
-      <origin xyz="0.0 0.0 0.0" rpy="0 0 0"/>
-      <mass value="0.0"/>
-      <inertia ixx="0.0" iyy="0.0" izz="0.0" ixy="0.0" iyz="0.0" ixz="0.0"/>
-    </inertial>
-  </link>
-  <link name="lens_focal_static_frame">
-    <inertial>
-      <origin xyz="0.0 0.0 0.0" rpy="0 0 0"/>
-      <mass value="0.0"/>
-      <inertia ixx="0.0" iyy="0.0" izz="0.0" ixy="0.0" iyz="0.0" ixz="0.0"/>
-    </inertial>
-  </link>
 <!--  JOINTS  .......................................................................................................-->
   <joint name="Boggie_right" type="revolute">
@@ -393,21 +371,3 @@
     <limit upper="0.698132" lower="-0.698132" effort="100" velocity="100"/>
   </joint>
-  <!--middle frame joint-->
-  <joint name="lens_frame_middle_joint" type="fixed">
-    <origin xyz="-0.2535  0.0 0.0" rpy="0 0 0"/>
-    <parent link="lens_Xrot_frame_1"/>
-    <child link="lens_frame_middle"/>
-  </joint>
-  <!--focal work frame joint-->
-  <joint name="lens_focal_work_frame_joint" type="fixed">
-    <origin xyz="0.0 0.0 -0.40" rpy="0 0 0"/>    <!-- posun v "z" je konstanta - zmenit -->
-    <parent link="lens_frame_middle"/>
-    <child link="lens_focal_work_frame"/>
-  </joint>
-  <!--focal static frame joint-->
-  <joint name="lens_focal_static_frame_joint" type="fixed">
-    <origin xyz="0.74 0.0 0.15" rpy="0 0 0"/>    <!-- posun v "x" a "z" je konstanta -(odcitat z robot-conf, ked sa vysunie sosovka)-->
-    <parent link="base_link"/>
-    <child link="lens_focal_static_frame"/>
-  </joint>
 </robot>

Commit message: rebase commits
updated Readme


Imu reading fix


added robot model


readme

updates


joint state publisher removed from launch


Odometry + joint state publisher

added robot model


renaming do->update


gitignore update cmake debug

File: ROS_ws/src/sPrinter_description/urdf/sPrinter.xacro (robot description, xacro)
@@ -285,4 +285,26 @@
     </collision>
   </link>
+  <!--  frame in the middle of the lens-->
+  <link name="lens_frame_middle">
+    <inertial>
+      <origin xyz="0.0 0.0 0.0" rpy="0 0 0"/>
+      <mass value="0.0"/>
+      <inertia ixx="0.0" iyy="0.0" izz="0.0" ixy="0.0" iyz="0.0" ixz="0.0"/>
+    </inertial>
+  </link>
+  <link name="lens_focal_work_frame">
+    <inertial>
+      <origin xyz="0.0 0.0 0.0" rpy="0 0 0"/>
+      <mass value="0.0"/>
+      <inertia ixx="0.0" iyy="0.0" izz="0.0" ixy="0.0" iyz="0.0" ixz="0.0"/>
+    </inertial>
+  </link>
+  <link name="lens_focal_static_frame">
+    <inertial>
+      <origin xyz="0.0 0.0 0.0" rpy="0 0 0"/>
+      <mass value="0.0"/>
+      <inertia ixx="0.0" iyy="0.0" izz="0.0" ixy="0.0" iyz="0.0" ixz="0.0"/>
+    </inertial>
+  </link>
 <!--  JOINTS  .......................................................................................................-->
   <joint name="Boggie_right" type="revolute">
@@ -371,3 +393,21 @@
     <limit upper="0.698132" lower="-0.698132" effort="100" velocity="100"/>
   </joint>
+  <!--middle frame joint-->
+  <joint name="lens_frame_middle_joint" type="fixed">
+    <origin xyz="-0.2535  0.0 0.0" rpy="0 0 0"/>
+    <parent link="lens_Xrot_frame_1"/>
+    <child link="lens_frame_middle"/>
+  </joint>
+  <!--focal work frame joint-->
+  <joint name="lens_focal_work_frame_joint" type="fixed">
+    <origin xyz="0.0 0.0 -0.40" rpy="0 0 0"/>    <!-- posun v "z" je konstanta - zmenit -->
+    <parent link="lens_frame_middle"/>
+    <child link="lens_focal_work_frame"/>
+  </joint>
+  <!--focal static frame joint-->
+  <joint name="lens_focal_static_frame_joint" type="fixed">
+    <origin xyz="0.74 0.0 0.15" rpy="0 0 0"/>    <!-- posun v "x" a "z" je konstanta -(odcitat z robot-conf, ked sa vysunie sosovka)-->
+    <parent link="base_link"/>
+    <child link="lens_focal_static_frame"/>
+  </joint>
 </robot>

Commit message: updated focal length

File: ROS_ws/src/sPrinter_description/urdf/sPrinter.xacro (robot description, xacro)
@@ -401,5 +401,6 @@
   <!--focal work frame joint-->
   <joint name="lens_focal_work_frame_joint" type="fixed">
-    <origin xyz="0.0 0.0 -0.40" rpy="0 0 0"/>    <!-- posun v "z" je konstanta - zmenit -->
+    <origin rpy="0 0 0" xyz="0.0 0.0 -0.50" />
+            <!-- z: ohniskova vzdialenost -->
     <parent link="lens_frame_middle"/>
     <child link="lens_focal_work_frame"/>
@@ -407,5 +408,7 @@
   <!--focal static frame joint-->
   <joint name="lens_focal_static_frame_joint" type="fixed">
-    <origin xyz="0.74 0.0 0.15" rpy="0 0 0"/>    <!-- posun v "x" a "z" je konstanta -(odcitat z robot-conf, ked sa vysunie sosovka)-->
+    <origin rpy="0 0 0" xyz="0.753764 0.0 0.05" />
+            <!-- z: 55cm - ohniskova vzdialenost = 5cm nad zemou-->
+            <!-- x: 0.753764 je pri 0.615m vysunuti sosovky v x (HOME) ... pod lens_midle frame-->
     <parent link="base_link"/>
     <child link="lens_focal_static_frame"/>

Commit message: changed to kdl ik solver, added idle2 robot pose

File: ROS_ws/src/sPrinter_description/urdf/sPrinter.xacro (robot description, xacro)
@@ -391,5 +391,5 @@
     <child link="lens_Xrot_frame_1"/>
     <axis xyz="1.0 -0.0 0.0"/>
-    <limit upper="0.698132" lower="-0.698132" effort="100" velocity="100"/>
+    <limit upper="1.2" lower="-1.2" effort="100" velocity="100"/>
   </joint>
   <!--middle frame joint-->

Commit message: refactor + enum in its own header

File: ROS_ws/src/sPrinter_description/urdf/sPrinter.xacro (robot description, xacro)
@@ -414,24 +414,3 @@
     <child link="lens_focal_static_frame"/>
   </joint>
-  <!--middle frame joint-->
-  <joint name="lens_frame_middle_joint" type="fixed">
-    <origin xyz="-0.2535  0.0 0.0" rpy="0 0 0"/>
-    <parent link="lens_Xrot_frame_1"/>
-    <child link="lens_frame_middle"/>
-  </joint>
-  <!--focal work frame joint-->
-  <joint name="lens_focal_work_frame_joint" type="fixed">
-    <origin rpy="0 0 0" xyz="0.0 0.0 -0.50" />
-            <!-- z: ohniskova vzdialenost -->
-    <parent link="lens_frame_middle"/>
-    <child link="lens_focal_work_frame"/>
-  </joint>
-  <!--focal static frame joint-->
-  <joint name="lens_focal_static_frame_joint" type="fixed">
-    <origin rpy="0 0 0" xyz="0.753764 0.0 0.05" />
-            <!-- z: 55cm - ohniskova vzdialenost = 5cm nad zemou-->
-            <!-- x: 0.753764 je pri 0.615m vysunuti sosovky v x (HOME) ... pod lens_midle frame-->
-    <parent link="base_link"/>
-    <child link="lens_focal_static_frame"/>
-  </joint>
 </robot>

Commit message: focal length to 55cm

File: ROS_ws/src/sPrinter_description/urdf/sPrinter.xacro (robot description, xacro)
@@ -401,5 +401,5 @@
   <!--focal work frame joint-->
   <joint name="lens_focal_work_frame_joint" type="fixed">
-    <origin rpy="0 0 0" xyz="0.0 0.0 -0.50" />
+    <origin rpy="0 0 0" xyz="0.0 0.0 -0.55" />
             <!-- z: ohniskova vzdialenost -->
     <parent link="lens_frame_middle"/>
@@ -408,6 +408,6 @@
   <!--focal static frame joint-->
   <joint name="lens_focal_static_frame_joint" type="fixed">
-    <origin rpy="0 0 0" xyz="0.753764 0.0 0.05" />
-            <!-- z: 55cm - ohniskova vzdialenost = 5cm nad zemou-->
+    <origin rpy="0 0 0" xyz="0.753764 0.0 -0.0" />
+            <!-- z: -55cm - ohniskova vzdialenost = 0cm nad rovinou zeme-->
             <!-- x: 0.753764 je pri 0.615m vysunuti sosovky v x (HOME) ... pod lens_midle frame-->
     <parent link="base_link"/>
