Commit message: `sPrinter_description`->`sprinter_description`
- removed obsolete files

File: ROS_ws/src/sprinter_description/urdf/sPrinter.xacro (robot description, xacro)
@@ -1,7 +1,7 @@
 <?xml version="1.0" ?>
 <robot name="sPrinter" xmlns:xacro="http://www.ros.org/wiki/xacro">
-  <xacro:include filename="$(find sPrinter_description)/urdf/materials.xacro" />
-  <xacro:include filename="$(find sPrinter_description)/urdf/sPrinter.trans" />
-  <xacro:include filename="$(find sPrinter_description)/urdf/sPrinter.gazebo" />
+  <xacro:include filename="$(find sprinter_description)/urdf/materials.xacro" />
+  <xacro:include filename="$(find sprinter_description)/urdf/sPrinter.trans" />
+  <xacro:include filename="$(find sprinter_description)/urdf/sPrinter.gazebo" />
   <!--  LINKS  ......................................................................................................-->
   <link name="base_link">
@@ -14,5 +14,5 @@
       <origin xyz="0 0 0" rpy="0 0 0"/>
       <geometry>
-        <mesh filename="package://sPrinter_description/meshes/base_link.stl" scale="0.001 0.001 0.001"/>
+        <mesh filename="package://sprinter_description/meshes/base_link.stl" scale="0.001 0.001 0.001"/>
       </geometry>
       <material name="silver"/>
@@ -21,5 +21,5 @@
       <origin xyz="0 0 0" rpy="0 0 0"/>
       <geometry>
-        <mesh filename="package://sPrinter_description/meshes/base_link.stl" scale="0.001 0.001 0.001"/>
+        <mesh filename="package://sprinter_description/meshes/base_link.stl" scale="0.001 0.001 0.001"/>
       </geometry>
     </collision>
@@ -34,5 +34,5 @@
       <origin xyz="0.26 0.22975 -0.21" rpy="0 0 0"/>
       <geometry>
-        <mesh filename="package://sPrinter_description/meshes/boggie_right_1.stl" scale="0.001 0.001 0.001"/>
+        <mesh filename="package://sprinter_description/meshes/boggie_right_1.stl" scale="0.001 0.001 0.001"/>
       </geometry>
       <material name="silver"/>
@@ -41,5 +41,5 @@
       <origin xyz="0.26 0.22975 -0.21" rpy="0 0 0"/>
       <geometry>
-        <mesh filename="package://sPrinter_description/meshes/boggie_right_1.stl" scale="0.001 0.001 0.001"/>
+        <mesh filename="package://sprinter_description/meshes/boggie_right_1.stl" scale="0.001 0.001 0.001"/>
       </geometry>
     </collision>
@@ -54,5 +54,5 @@
       <origin xyz="0.26 -0.22975 -0.21" rpy="0 0 0"/>
       <geometry>
-        <mesh filename="package://sPrinter_description/meshes/boggie_left_1.stl" scale="0.001 0.001 0.001"/>
+        <mesh filename="package://sprinter_description/meshes/boggie_left_1.stl" scale="0.001 0.001 0.001"/>
       </geometry>
       <material name="silver"/>
@@ -61,5 +61,5 @@
       <origin xyz="0.26 -0.22975 -0.21" rpy="0 0 0"/>
       <geometry>
-        <mesh filename="package://sPrinter_description/meshes/boggie_left_1.stl" scale="0.001 0.001 0.001"/>
+        <mesh filename="package://sprinter_description/meshes/boggie_left_1.stl" scale="0.001 0.001 0.001"/>
       </geometry>
     </collision>
@@ -74,5 +74,5 @@
       <origin xyz="-0.42 0.38275 -0.09" rpy="0 0 0"/>
       <geometry>
-        <mesh filename="package://sPrinter_description/meshes/wheel_right_front_1.stl" scale="0.001 0.001 0.001"/>
+        <mesh filename="package://sprinter_description/meshes/wheel_right_front_1.stl" scale="0.001 0.001 0.001"/>
       </geometry>
       <material name="silver"/>
@@ -81,5 +81,5 @@
       <origin xyz="-0.42 0.38275 -0.09" rpy="0 0 0"/>
       <geometry>
-        <mesh filename="package://sPrinter_description/meshes/wheel_right_front_1.stl" scale="0.001 0.001 0.001"/>
+        <mesh filename="package://sprinter_description/meshes/wheel_right_front_1.stl" scale="0.001 0.001 0.001"/>
       </geometry>
     </collision>
@@ -94,5 +94,5 @@
       <origin xyz="0.0 0.40375 -0.09" rpy="0 0 0"/>
       <geometry>
-        <mesh filename="package://sPrinter_description/meshes/wheel_right_middle_1.stl" scale="0.001 0.001 0.001"/>
+        <mesh filename="package://sprinter_description/meshes/wheel_right_middle_1.stl" scale="0.001 0.001 0.001"/>
       </geometry>
       <material name="silver"/>
@@ -101,5 +101,5 @@
       <origin xyz="0.0 0.40375 -0.09" rpy="0 0 0"/>
       <geometry>
-        <mesh filename="package://sPrinter_description/meshes/wheel_right_middle_1.stl" scale="0.001 0.001 0.001"/>
+        <mesh filename="package://sprinter_description/meshes/wheel_right_middle_1.stl" scale="0.001 0.001 0.001"/>
       </geometry>
     </collision>
@@ -114,5 +114,5 @@
       <origin xyz="0.42 0.40375 -0.09" rpy="0 0 0"/>
       <geometry>
-        <mesh filename="package://sPrinter_description/meshes/wheel_right_rear__1.stl" scale="0.001 0.001 0.001"/>
+        <mesh filename="package://sprinter_description/meshes/wheel_right_rear__1.stl" scale="0.001 0.001 0.001"/>
       </geometry>
       <material name="silver"/>
@@ -121,5 +121,5 @@
       <origin xyz="0.42 0.40375 -0.09" rpy="0 0 0"/>
       <geometry>
-        <mesh filename="package://sPrinter_description/meshes/wheel_right_rear__1.stl" scale="0.001 0.001 0.001"/>
+        <mesh filename="package://sprinter_description/meshes/wheel_right_rear__1.stl" scale="0.001 0.001 0.001"/>
       </geometry>
     </collision>
@@ -134,5 +134,5 @@
       <origin xyz="-0.42 -0.38275 -0.09" rpy="0 0 0"/>
       <geometry>
-        <mesh filename="package://sPrinter_description/meshes/wheel_left_front_1.stl" scale="0.001 0.001 0.001"/>
+        <mesh filename="package://sprinter_description/meshes/wheel_left_front_1.stl" scale="0.001 0.001 0.001"/>
       </geometry>
       <material name="silver"/>
@@ -141,5 +141,5 @@
       <origin xyz="-0.42 -0.38275 -0.09" rpy="0 0 0"/>
       <geometry>
-        <mesh filename="package://sPrinter_description/meshes/wheel_left_front_1.stl" scale="0.001 0.001 0.001"/>
+        <mesh filename="package://sprinter_description/meshes/wheel_left_front_1.stl" scale="0.001 0.001 0.001"/>
       </geometry>
     </collision>
@@ -154,5 +154,5 @@
       <origin xyz="-0.0 -0.40375 -0.09" rpy="0 0 0"/>
       <geometry>
-        <mesh filename="package://sPrinter_description/meshes/wheel_left_middle_1.stl" scale="0.001 0.001 0.001"/>
+        <mesh filename="package://sprinter_description/meshes/wheel_left_middle_1.stl" scale="0.001 0.001 0.001"/>
       </geometry>
       <material name="silver"/>
@@ -161,5 +161,5 @@
       <origin xyz="-0.0 -0.40375 -0.09" rpy="0 0 0"/>
       <geometry>
-        <mesh filename="package://sPrinter_description/meshes/wheel_left_middle_1.stl" scale="0.001 0.001 0.001"/>
+        <mesh filename="package://sprinter_description/meshes/wheel_left_middle_1.stl" scale="0.001 0.001 0.001"/>
       </geometry>
     </collision>
@@ -174,5 +174,5 @@
       <origin xyz="0.42 -0.40375 -0.09" rpy="0 0 0"/>
       <geometry>
-        <mesh filename="package://sPrinter_description/meshes/wheel_left_rear_1.stl" scale="0.001 0.001 0.001"/>
+        <mesh filename="package://sprinter_description/meshes/wheel_left_rear_1.stl" scale="0.001 0.001 0.001"/>
       </geometry>
       <material name="silver"/>
@@ -181,5 +181,5 @@
       <origin xyz="0.42 -0.40375 -0.09" rpy="0 0 0"/>
       <geometry>
-        <mesh filename="package://sPrinter_description/meshes/wheel_left_rear_1.stl" scale="0.001 0.001 0.001"/>
+        <mesh filename="package://sprinter_description/meshes/wheel_left_rear_1.stl" scale="0.001 0.001 0.001"/>
       </geometry>
     </collision>
@@ -194,5 +194,5 @@
       <origin xyz="0.0 0.0 -0.31" rpy="0 0 0"/>
       <geometry>
-        <mesh filename="package://sPrinter_description/meshes/main_frame_1.stl" scale="0.001 0.001 0.001"/>
+        <mesh filename="package://sprinter_description/meshes/main_frame_1.stl" scale="0.001 0.001 0.001"/>
       </geometry>
       <material name="silver"/>
@@ -201,5 +201,5 @@
       <origin xyz="0.0 0.0 -0.31" rpy="0 0 0"/>
       <geometry>
-        <mesh filename="package://sPrinter_description/meshes/main_frame_1.stl" scale="0.001 0.001 0.001"/>
+        <mesh filename="package://sprinter_description/meshes/main_frame_1.stl" scale="0.001 0.001 0.001"/>
       </geometry>
     </collision>
@@ -214,5 +214,5 @@
       <origin xyz="-0.1445 0.020515 -0.453" rpy="0 0 0"/>
       <geometry>
-        <mesh filename="package://sPrinter_description/meshes/lens_Ylin_frame_1.stl" scale="0.001 0.001 0.001"/>
+        <mesh filename="package://sprinter_description/meshes/lens_Ylin_frame_1.stl" scale="0.001 0.001 0.001"/>
       </geometry>
       <material name="silver"/>
@@ -221,5 +221,5 @@
       <origin xyz="-0.1445 0.020515 -0.453" rpy="0 0 0"/>
       <geometry>
-        <mesh filename="package://sPrinter_description/meshes/lens_Ylin_frame_1.stl" scale="0.001 0.001 0.001"/>
+        <mesh filename="package://sprinter_description/meshes/lens_Ylin_frame_1.stl" scale="0.001 0.001 0.001"/>
       </geometry>
     </collision>
@@ -234,5 +234,5 @@
       <origin xyz="0.2502 0.0 -0.49414" rpy="0 0 0"/>
       <geometry>
-        <mesh filename="package://sPrinter_description/meshes/lens_Xlin_frame_1.stl" scale="0.001 0.001 0.001"/>
+        <mesh filename="package://sprinter_description/meshes/lens_Xlin_frame_1.stl" scale="0.001 0.001 0.001"/>
       </geometry>
       <material name="silver"/>
@@ -241,5 +241,5 @@
       <origin xyz="0.2502 0.0 -0.49414" rpy="0 0 0"/>
       <geometry>
-        <mesh filename="package://sPrinter_description/meshes/lens_Xlin_frame_1.stl" scale="0.001 0.001 0.001"/>
+        <mesh filename="package://sprinter_description/meshes/lens_Xlin_frame_1.stl" scale="0.001 0.001 0.001"/>
       </geometry>
     </collision>
@@ -254,5 +254,5 @@
       <origin xyz="-0.144866 -0.270552 -0.528953" rpy="0 0 0"/>
       <geometry>
-        <mesh filename="package://sPrinter_description/meshes/lens_Yrot_frame__1.stl" scale="0.001 0.001 0.001"/>
+        <mesh filename="package://sprinter_description/meshes/lens_Yrot_frame__1.stl" scale="0.001 0.001 0.001"/>
       </geometry>
       <material name="silver"/>
@@ -261,5 +261,5 @@
       <origin xyz="-0.144866 -0.270552 -0.528953" rpy="0 0 0"/>
       <geometry>
-        <mesh filename="package://sPrinter_description/meshes/lens_Yrot_frame__1.stl" scale="0.001 0.001 0.001"/>
+        <mesh filename="package://sprinter_description/meshes/lens_Yrot_frame__1.stl" scale="0.001 0.001 0.001"/>
       </geometry>
     </collision>
@@ -274,5 +274,5 @@
       <origin xyz="-0.392366 8.1e-05 -0.552581" rpy="0 0 0"/>
       <geometry>
-        <mesh filename="package://sPrinter_description/meshes/lens_Xrot_frame_1.stl" scale="0.001 0.001 0.001"/>
+        <mesh filename="package://sprinter_description/meshes/lens_Xrot_frame_1.stl" scale="0.001 0.001 0.001"/>
       </geometry>
       <material name="silver"/>
@@ -281,5 +281,5 @@
       <origin xyz="-0.392366 8.1e-05 -0.552581" rpy="0 0 0"/>
       <geometry>
-        <mesh filename="package://sPrinter_description/meshes/lens_Xrot_frame_1.stl" scale="0.001 0.001 0.001"/>
+        <mesh filename="package://sprinter_description/meshes/lens_Xrot_frame_1.stl" scale="0.001 0.001 0.001"/>
       </geometry>
     </collision>
