Commit message: removed __1 and _1

File: ROS_ws/src/sprinter_description/urdf/sPrinter.xacro (robot description, xacro)
@@ -25,5 +25,5 @@
     </collision>
   </link>
-  <link name="boggie_right_1">
+  <link name="boggie_right">
     <inertial>
       <origin xyz="0.04608835670723324 -0.05868381694977415 -0.08782934708885383" rpy="0 0 0"/>
@@ -34,5 +34,5 @@
       <origin xyz="0.26 0.22975 -0.21" rpy="0 0 0"/>
       <geometry>
-        <mesh filename="package://sprinter_description/meshes/boggie_right_1.stl" scale="0.001 0.001 0.001"/>
+        <mesh filename="package://sprinter_description/meshes/boggie_right.stl" scale="0.001 0.001 0.001"/>
       </geometry>
       <material name="silver"/>
@@ -41,9 +41,9 @@
       <origin xyz="0.26 0.22975 -0.21" rpy="0 0 0"/>
       <geometry>
-        <mesh filename="package://sprinter_description/meshes/boggie_right_1.stl" scale="0.001 0.001 0.001"/>
-      </geometry>
-    </collision>
-  </link>
-  <link name="boggie_left_1">
+        <mesh filename="package://sprinter_description/meshes/boggie_right.stl" scale="0.001 0.001 0.001"/>
+      </geometry>
+    </collision>
+  </link>
+  <link name="boggie_left">
     <inertial>
       <origin xyz="0.04608852267144553 0.05868381722034843 -0.0878295588540255" rpy="0 0 0"/>
@@ -54,5 +54,5 @@
       <origin xyz="0.26 -0.22975 -0.21" rpy="0 0 0"/>
       <geometry>
-        <mesh filename="package://sprinter_description/meshes/boggie_left_1.stl" scale="0.001 0.001 0.001"/>
+        <mesh filename="package://sprinter_description/meshes/boggie_left.stl" scale="0.001 0.001 0.001"/>
       </geometry>
       <material name="silver"/>
@@ -61,9 +61,9 @@
       <origin xyz="0.26 -0.22975 -0.21" rpy="0 0 0"/>
       <geometry>
-        <mesh filename="package://sprinter_description/meshes/boggie_left_1.stl" scale="0.001 0.001 0.001"/>
-      </geometry>
-    </collision>
-  </link>
-  <link name="wheel_right_front_1">
+        <mesh filename="package://sprinter_description/meshes/boggie_left.stl" scale="0.001 0.001 0.001"/>
+      </geometry>
+    </collision>
+  </link>
+  <link name="wheel_right_front">
     <inertial>
       <origin xyz="-2.2157215140428121e-07 0.049038331285879255 -5.319570878098423e-07" rpy="0 0 0"/>
@@ -74,5 +74,5 @@
       <origin xyz="-0.42 0.38275 -0.09" rpy="0 0 0"/>
       <geometry>
-        <mesh filename="package://sprinter_description/meshes/wheel_right_front_1.stl" scale="0.001 0.001 0.001"/>
+        <mesh filename="package://sprinter_description/meshes/wheel_right_front.stl" scale="0.001 0.001 0.001"/>
       </geometry>
       <material name="silver"/>
@@ -81,9 +81,9 @@
       <origin xyz="-0.42 0.38275 -0.09" rpy="0 0 0"/>
       <geometry>
-        <mesh filename="package://sprinter_description/meshes/wheel_right_front_1.stl" scale="0.001 0.001 0.001"/>
-      </geometry>
-    </collision>
-  </link>
-  <link name="wheel_right_middle_1">
+        <mesh filename="package://sprinter_description/meshes/wheel_right_front.stl" scale="0.001 0.001 0.001"/>
+      </geometry>
+    </collision>
+  </link>
+  <link name="wheel_right_middle">
     <inertial>
       <origin xyz="-2.441464656044445e-07 0.049038331285878034 -1.2471173249650747e-07" rpy="0 0 0"/>
@@ -94,5 +94,5 @@
       <origin xyz="0.0 0.40375 -0.09" rpy="0 0 0"/>
       <geometry>
-        <mesh filename="package://sprinter_description/meshes/wheel_right_middle_1.stl" scale="0.001 0.001 0.001"/>
+        <mesh filename="package://sprinter_description/meshes/wheel_right_middle.stl" scale="0.001 0.001 0.001"/>
       </geometry>
       <material name="silver"/>
@@ -101,9 +101,9 @@
       <origin xyz="0.0 0.40375 -0.09" rpy="0 0 0"/>
       <geometry>
-        <mesh filename="package://sprinter_description/meshes/wheel_right_middle_1.stl" scale="0.001 0.001 0.001"/>
-      </geometry>
-    </collision>
-  </link>
-  <link name="wheel_right_rear__1">
+        <mesh filename="package://sprinter_description/meshes/wheel_right_middle.stl" scale="0.001 0.001 0.001"/>
+      </geometry>
+    </collision>
+  </link>
+  <link name="wheel_right_rear">
     <inertial>
       <origin xyz="-2.4414526850202733e-07 0.04903833128586854 4.1045225383784523e-07" rpy="0 0 0"/>
@@ -114,5 +114,5 @@
       <origin xyz="0.42 0.40375 -0.09" rpy="0 0 0"/>
       <geometry>
-        <mesh filename="package://sprinter_description/meshes/wheel_right_rear__1.stl" scale="0.001 0.001 0.001"/>
+        <mesh filename="package://sprinter_description/meshes/wheel_right_rear.stl" scale="0.001 0.001 0.001"/>
       </geometry>
       <material name="silver"/>
@@ -121,9 +121,9 @@
       <origin xyz="0.42 0.40375 -0.09" rpy="0 0 0"/>
       <geometry>
-        <mesh filename="package://sprinter_description/meshes/wheel_right_rear__1.stl" scale="0.001 0.001 0.001"/>
-      </geometry>
-    </collision>
-  </link>
-  <link name="wheel_left_front_1">
+        <mesh filename="package://sprinter_description/meshes/wheel_right_rear.stl" scale="0.001 0.001 0.001"/>
+      </geometry>
+    </collision>
+  </link>
+  <link name="wheel_left_front">
     <inertial>
       <origin xyz="-1.7782965933133e-08 -0.04903833128669849 -7.65968576066367e-08" rpy="0 0 0"/>
@@ -134,5 +134,5 @@
       <origin xyz="-0.42 -0.38275 -0.09" rpy="0 0 0"/>
       <geometry>
-        <mesh filename="package://sprinter_description/meshes/wheel_left_front_1.stl" scale="0.001 0.001 0.001"/>
+        <mesh filename="package://sprinter_description/meshes/wheel_left_front.stl" scale="0.001 0.001 0.001"/>
       </geometry>
       <material name="silver"/>
@@ -141,9 +141,9 @@
       <origin xyz="-0.42 -0.38275 -0.09" rpy="0 0 0"/>
       <geometry>
-        <mesh filename="package://sprinter_description/meshes/wheel_left_front_1.stl" scale="0.001 0.001 0.001"/>
-      </geometry>
-    </collision>
-  </link>
-  <link name="wheel_left_middle_1">
+        <mesh filename="package://sprinter_description/meshes/wheel_left_front.stl" scale="0.001 0.001 0.001"/>
+      </geometry>
+    </collision>
+  </link>
+  <link name="wheel_left_middle">
     <inertial>
       <origin xyz="1.038819750736053e-06 -0.049038331286717474 0.00010982563519425226" rpy="0 0 0"/>
@@ -154,5 +154,5 @@
       <origin xyz="-0.0 -0.40375 -0.09" rpy="0 0 0"/>
       <geometry>
-        <mesh filename="package://sprinter_description/meshes/wheel_left_middle_1.stl" scale="0.001 0.001 0.001"/>
+        <mesh filename="package://sprinter_description/meshes/wheel_left_middle.stl" scale="0.001 0.001 0.001"/>
       </geometry>
       <material name="silver"/>
@@ -161,9 +161,9 @@
       <origin xyz="-0.0 -0.40375 -0.09" rpy="0 0 0"/>
       <geometry>
-        <mesh filename="package://sprinter_description/meshes/wheel_left_middle_1.stl" scale="0.001 0.001 0.001"/>
-      </geometry>
-    </collision>
-  </link>
-  <link name="wheel_left_rear_1">
+        <mesh filename="package://sprinter_description/meshes/wheel_left_middle.stl" scale="0.001 0.001 0.001"/>
+      </geometry>
+    </collision>
+  </link>
+  <link name="wheel_left_rear">
     <inertial>
       <origin xyz="1.0388197915767172e-06 -0.04903833128671531 0.00010972160107960982" rpy="0 0 0"/>
@@ -174,5 +174,5 @@
       <origin xyz="0.42 -0.40375 -0.09" rpy="0 0 0"/>
       <geometry>
-        <mesh filename="package://sprinter_description/meshes/wheel_left_rear_1.stl" scale="0.001 0.001 0.001"/>
+        <mesh filename="package://sprinter_description/meshes/wheel_left_rear.stl" scale="0.001 0.001 0.001"/>
       </geometry>
       <material name="silver"/>
@@ -181,9 +181,9 @@
       <origin xyz="0.42 -0.40375 -0.09" rpy="0 0 0"/>
       <geometry>
-        <mesh filename="package://sprinter_description/meshes/wheel_left_rear_1.stl" scale="0.001 0.001 0.001"/>
-      </geometry>
-    </collision>
-  </link>
-  <link name="main_frame_1">
+        <mesh filename="package://sprinter_description/meshes/wheel_left_rear.stl" scale="0.001 0.001 0.001"/>
+      </geometry>
+    </collision>
+  </link>
+  <link name="main_frame">
     <inertial>
       <origin xyz="-0.08748571926603223 0.002858790568392067 -0.009190179413522459" rpy="0 0 0"/>
@@ -194,5 +194,5 @@
       <origin xyz="0.0 0.0 -0.31" rpy="0 0 0"/>
       <geometry>
-        <mesh filename="package://sprinter_description/meshes/main_frame_1.stl" scale="0.001 0.001 0.001"/>
+        <mesh filename="package://sprinter_description/meshes/main_frame.stl" scale="0.001 0.001 0.001"/>
       </geometry>
       <material name="silver"/>
@@ -201,9 +201,9 @@
       <origin xyz="0.0 0.0 -0.31" rpy="0 0 0"/>
       <geometry>
-        <mesh filename="package://sprinter_description/meshes/main_frame_1.stl" scale="0.001 0.001 0.001"/>
-      </geometry>
-    </collision>
-  </link>
-  <link name="lens_Ylin_frame_1">
+        <mesh filename="package://sprinter_description/meshes/main_frame.stl" scale="0.001 0.001 0.001"/>
+      </geometry>
+    </collision>
+  </link>
+  <link name="lens_Ylin_frame">
     <inertial>
       <origin xyz="-0.19050492237401995 0.01911574728140262 0.050354275554037764" rpy="0 0 0"/>
@@ -214,5 +214,5 @@
       <origin xyz="-0.1445 0.020515 -0.453" rpy="0 0 0"/>
       <geometry>
-        <mesh filename="package://sprinter_description/meshes/lens_Ylin_frame_1.stl" scale="0.001 0.001 0.001"/>
+        <mesh filename="package://sprinter_description/meshes/lens_Ylin_frame.stl" scale="0.001 0.001 0.001"/>
       </geometry>
       <material name="silver"/>
@@ -221,9 +221,9 @@
       <origin xyz="-0.1445 0.020515 -0.453" rpy="0 0 0"/>
       <geometry>
-        <mesh filename="package://sprinter_description/meshes/lens_Ylin_frame_1.stl" scale="0.001 0.001 0.001"/>
-      </geometry>
-    </collision>
-  </link>
-  <link name="lens_Xlin_frame_1">
+        <mesh filename="package://sprinter_description/meshes/lens_Ylin_frame.stl" scale="0.001 0.001 0.001"/>
+      </geometry>
+    </collision>
+  </link>
+  <link name="lens_Xlin_frame">
     <inertial>
       <origin xyz="0.23595566779369742 0.13671241587093597 0.03333844333172431" rpy="0 0 0"/>
@@ -234,5 +234,5 @@
       <origin xyz="0.2502 0.0 -0.49414" rpy="0 0 0"/>
       <geometry>
-        <mesh filename="package://sprinter_description/meshes/lens_Xlin_frame_1.stl" scale="0.001 0.001 0.001"/>
+        <mesh filename="package://sprinter_description/meshes/lens_Xlin_frame.stl" scale="0.001 0.001 0.001"/>
       </geometry>
       <material name="silver"/>
@@ -241,9 +241,9 @@
       <origin xyz="0.2502 0.0 -0.49414" rpy="0 0 0"/>
       <geometry>
-        <mesh filename="package://sprinter_description/meshes/lens_Xlin_frame_1.stl" scale="0.001 0.001 0.001"/>
-      </geometry>
-    </collision>
-  </link>
-  <link name="lens_Yrot_frame__1">
+        <mesh filename="package://sprinter_description/meshes/lens_Xlin_frame.stl" scale="0.001 0.001 0.001"/>
+      </geometry>
+    </collision>
+  </link>
+  <link name="lens_Yrot_frame">
     <inertial>
       <origin xyz="0.15610000473558938 -0.28034931010215036 0.01290803779832872" rpy="0 0 0"/>
@@ -254,5 +254,5 @@
       <origin xyz="-0.144866 -0.270552 -0.528953" rpy="0 0 0"/>
       <geometry>
-        <mesh filename="package://sprinter_description/meshes/lens_Yrot_frame__1.stl" scale="0.001 0.001 0.001"/>
+        <mesh filename="package://sprinter_description/meshes/lens_Yrot_frame.stl" scale="0.001 0.001 0.001"/>
       </geometry>
       <material name="silver"/>
@@ -261,9 +261,9 @@
       <origin xyz="-0.144866 -0.270552 -0.528953" rpy="0 0 0"/>
       <geometry>
-        <mesh filename="package://sprinter_description/meshes/lens_Yrot_frame__1.stl" scale="0.001 0.001 0.001"/>
-      </geometry>
-    </collision>
-  </link>
-  <link name="lens_Xrot_frame_1">
+        <mesh filename="package://sprinter_description/meshes/lens_Yrot_frame.stl" scale="0.001 0.001 0.001"/>
+      </geometry>
+    </collision>
+  </link>
+  <link name="lens_Xrot_frame">
     <inertial>
       <origin xyz="-0.2533217422271652 7.584721687383723e-06 0.0013476837862036462" rpy="0 0 0"/>
@@ -274,5 +274,5 @@
       <origin xyz="-0.392366 8.1e-05 -0.552581" rpy="0 0 0"/>
       <geometry>
-        <mesh filename="package://sprinter_description/meshes/lens_Xrot_frame_1.stl" scale="0.001 0.001 0.001"/>
+        <mesh filename="package://sprinter_description/meshes/lens_Xrot_frame.stl" scale="0.001 0.001 0.001"/>
       </geometry>
       <material name="silver"/>
@@ -281,5 +281,5 @@
       <origin xyz="-0.392366 8.1e-05 -0.552581" rpy="0 0 0"/>
       <geometry>
-        <mesh filename="package://sprinter_description/meshes/lens_Xrot_frame_1.stl" scale="0.001 0.001 0.001"/>
+        <mesh filename="package://sprinter_description/meshes/lens_Xrot_frame.stl" scale="0.001 0.001 0.001"/>
       </geometry>
     </collision>
@@ -311,5 +311,5 @@
     <origin xyz="-0.26 -0.22975 0.21" rpy="0 0 0"/>
     <parent link="base_link"/>
-    <child link="boggie_right_1"/>
+    <child link="boggie_right"/>
     <axis xyz="-0.0 1.0 0.0"/>
     <limit upper="0.523599" lower="-0.523599" effort="100" velocity="100"/>
@@ -318,5 +318,5 @@
     <origin xyz="-0.26 0.22975 0.21" rpy="0 0 0"/>
     <parent link="base_link"/>
-    <child link="boggie_left_1"/>
+    <child link="boggie_left"/>
     <axis xyz="0.0 1.0 0.0"/>
     <limit upper="0.523599" lower="-0.523599" effort="100" velocity="100"/>
@@ -325,17 +325,17 @@
     <origin xyz="0.42 -0.38275 0.09" rpy="0 0 0"/>
     <parent link="base_link"/>
-    <child link="wheel_right_front_1"/>
+    <child link="wheel_right_front"/>
     <axis xyz="0.0 1.0 0.0"/>
   </joint>
   <joint name="Wheel_right_middle" type="continuous">
     <origin xyz="0.26 -0.174 -0.12" rpy="0 0 0"/>
-    <parent link="boggie_right_1"/>
-    <child link="wheel_right_middle_1"/>
+    <parent link="boggie_right"/>
+    <child link="wheel_right_middle"/>
     <axis xyz="0.0 1.0 0.0"/>
   </joint>
   <joint name="Wheel_right_rear" type="continuous">
     <origin xyz="-0.16 -0.174 -0.12" rpy="0 0 0"/>
-    <parent link="boggie_right_1"/>
-    <child link="wheel_right_rear__1"/>
+    <parent link="boggie_right"/>
+    <child link="wheel_right_rear"/>
     <axis xyz="0.0 1.0 0.0"/>
   </joint>
@@ -343,17 +343,17 @@
     <origin xyz="0.42 0.38275 0.09" rpy="0 0 0"/>
     <parent link="base_link"/>
-    <child link="wheel_left_front_1"/>
+    <child link="wheel_left_front"/>
     <axis xyz="0.0 1.0 0.0"/>
   </joint>
   <joint name="Wheel_left_middle" type="continuous">
     <origin xyz="0.26 0.174 -0.12" rpy="0 0 0"/>
-    <parent link="boggie_left_1"/>
-    <child link="wheel_left_middle_1"/>
+    <parent link="boggie_left"/>
+    <child link="wheel_left_middle"/>
     <axis xyz="0.0 1.0 0.0"/>
   </joint>
   <joint name="Wheel_left_rear" type="continuous">
     <origin xyz="-0.16 0.174 -0.12" rpy="0 0 0"/>
-    <parent link="boggie_left_1"/>
-    <child link="wheel_left_rear_1"/>
+    <parent link="boggie_left"/>
+    <child link="wheel_left_rear"/>
     <axis xyz="0.0 1.0 0.0"/>
   </joint>
@@ -361,5 +361,5 @@
     <origin xyz="0.0 0.0 0.31" rpy="0 0 0"/>
     <parent link="base_link"/>
-    <child link="main_frame_1"/>
+    <child link="main_frame"/>
     <axis xyz="-0.0 1.0 0.0"/>
     <limit upper="0.523599" lower="-0.523599" effort="100" velocity="100"/>
@@ -367,6 +367,6 @@
   <joint name="Lens_Y_axis_trans" type="prismatic">
     <origin xyz="0.1445 -0.020515 0.143" rpy="0 0 0"/>
-    <parent link="main_frame_1"/>
-    <child link="lens_Ylin_frame_1"/>
+    <parent link="main_frame"/>
+    <child link="lens_Ylin_frame"/>
     <axis xyz="0.0 1.0 0.0"/>
     <limit upper="0.15" lower="-0.12" effort="100" velocity="100"/>
@@ -374,6 +374,6 @@
   <joint name="Lens_X_axis_trans" type="prismatic">
     <origin xyz="-0.3947 0.020515 0.04114" rpy="0 0 0"/>
-    <parent link="lens_Ylin_frame_1"/>
-    <child link="lens_Xlin_frame_1"/>
+    <parent link="lens_Ylin_frame"/>
+    <child link="lens_Xlin_frame"/>
     <axis xyz="1.0 -0.0 0.0"/>
     <limit upper="0.65" lower="0.0" effort="100" velocity="100"/>
@@ -381,6 +381,6 @@
   <joint name="Lens_Y_axis_rot" type="revolute">
     <origin xyz="0.395066 0.270552 0.034813" rpy="0 0 0"/>
-    <parent link="lens_Xlin_frame_1"/>
-    <child link="lens_Yrot_frame__1"/>
+    <parent link="lens_Xlin_frame"/>
+    <child link="lens_Yrot_frame"/>
     <axis xyz="0.0 0.999999 0.001376"/>
     <limit upper="0.698132" lower="-0.698132" effort="100" velocity="100"/>
@@ -388,6 +388,6 @@
   <joint name="Lens_X_axis_rot" type="revolute">
     <origin xyz="0.2475 -0.270633 0.023628" rpy="0 0 0"/>
-    <parent link="lens_Yrot_frame__1"/>
-    <child link="lens_Xrot_frame_1"/>
+    <parent link="lens_Yrot_frame"/>
+    <child link="lens_Xrot_frame"/>
     <axis xyz="1.0 -0.0 0.0"/>
     <limit upper="1.2" lower="-1.2" effort="100" velocity="100"/>
@@ -396,5 +396,5 @@
   <joint name="lens_frame_middle_joint" type="fixed">
     <origin xyz="-0.2535  0.0 0.0" rpy="0 0 0"/>
-    <parent link="lens_Xrot_frame_1"/>
+    <parent link="lens_Xrot_frame"/>
     <child link="lens_frame_middle"/>
   </joint>
