Commit message: _frame removed

File: ROS_ws/src/sprinter_description/urdf/sPrinter.urdf (robot description, URDF)
Before this commit: robot sPrinter, 17 links, 16 joints
Links:
- removed link lens_Xlin_frame
- removed link lens_Xrot_frame
- removed link lens_Ylin_frame
- removed link lens_Yrot_frame
- added link lens_Xlin, mass 1.8074023885886255; collision mesh filename=package://sprinter_description/meshes/lens_Xlin.stl scale=0.001 0.001 0.001; visual mesh filename=package://sprinter_description/meshes/lens_Xlin.stl scale=0.001 0.001 0.001
- added link lens_Xrot, mass 6.552542872975625; collision mesh filename=package://sprinter_description/meshes/lens_Xrot.stl scale=0.001 0.001 0.001; visual mesh filename=package://sprinter_description/meshes/lens_Xrot.stl scale=0.001 0.001 0.001
- added link lens_Ylin, mass 8.115658394698128; collision mesh filename=package://sprinter_description/meshes/lens_Ylin.stl scale=0.001 0.001 0.001; visual mesh filename=package://sprinter_description/meshes/lens_Ylin.stl scale=0.001 0.001 0.001
- added link lens_Yrot, mass 1.6400641565943115; collision mesh filename=package://sprinter_description/meshes/lens_Yrot.stl scale=0.001 0.001 0.001; visual mesh filename=package://sprinter_description/meshes/lens_Yrot.stl scale=0.001 0.001 0.001
Joints:
- joint Lens_X_axis_rot: child lens_Xrot_frame -> lens_Xrot; parent lens_Yrot_frame -> lens_Yrot
- joint Lens_X_axis_trans: child lens_Xlin_frame -> lens_Xlin; parent lens_Ylin_frame -> lens_Ylin
- joint Lens_Y_axis_rot: child lens_Yrot_frame -> lens_Yrot; parent lens_Xlin_frame -> lens_Xlin
- joint Lens_Y_axis_trans: child lens_Ylin_frame -> lens_Ylin
- joint lens_frame_middle_joint: parent lens_Xrot_frame -> lens_Xrot

File: ROS_ws/src/sprinter_description/urdf/sPrinter.xacro (robot description, xacro)
@@ -205,5 +205,5 @@
     </collision>
   </link>
-  <link name="lens_Ylin_frame">
+  <link name="lens_Ylin">
     <inertial>
       <origin xyz="-0.19050492237401995 0.01911574728140262 0.050354275554037764" rpy="0 0 0"/>
@@ -214,5 +214,5 @@
       <origin xyz="-0.1445 0.020515 -0.453" rpy="0 0 0"/>
       <geometry>
-        <mesh filename="package://sprinter_description/meshes/lens_Ylin_frame.stl" scale="0.001 0.001 0.001"/>
+        <mesh filename="package://sprinter_description/meshes/lens_Ylin.stl" scale="0.001 0.001 0.001"/>
       </geometry>
       <material name="silver"/>
@@ -221,9 +221,9 @@
       <origin xyz="-0.1445 0.020515 -0.453" rpy="0 0 0"/>
       <geometry>
-        <mesh filename="package://sprinter_description/meshes/lens_Ylin_frame.stl" scale="0.001 0.001 0.001"/>
-      </geometry>
-    </collision>
-  </link>
-  <link name="lens_Xlin_frame">
+        <mesh filename="package://sprinter_description/meshes/lens_Ylin.stl" scale="0.001 0.001 0.001"/>
+      </geometry>
+    </collision>
+  </link>
+  <link name="lens_Xlin">
     <inertial>
       <origin xyz="0.23595566779369742 0.13671241587093597 0.03333844333172431" rpy="0 0 0"/>
@@ -234,5 +234,5 @@
       <origin xyz="0.2502 0.0 -0.49414" rpy="0 0 0"/>
       <geometry>
-        <mesh filename="package://sprinter_description/meshes/lens_Xlin_frame.stl" scale="0.001 0.001 0.001"/>
+        <mesh filename="package://sprinter_description/meshes/lens_Xlin.stl" scale="0.001 0.001 0.001"/>
       </geometry>
       <material name="silver"/>
@@ -241,9 +241,9 @@
       <origin xyz="0.2502 0.0 -0.49414" rpy="0 0 0"/>
       <geometry>
-        <mesh filename="package://sprinter_description/meshes/lens_Xlin_frame.stl" scale="0.001 0.001 0.001"/>
-      </geometry>
-    </collision>
-  </link>
-  <link name="lens_Yrot_frame">
+        <mesh filename="package://sprinter_description/meshes/lens_Xlin.stl" scale="0.001 0.001 0.001"/>
+      </geometry>
+    </collision>
+  </link>
+  <link name="lens_Yrot">
     <inertial>
       <origin xyz="0.15610000473558938 -0.28034931010215036 0.01290803779832872" rpy="0 0 0"/>
@@ -254,5 +254,5 @@
       <origin xyz="-0.144866 -0.270552 -0.528953" rpy="0 0 0"/>
       <geometry>
-        <mesh filename="package://sprinter_description/meshes/lens_Yrot_frame.stl" scale="0.001 0.001 0.001"/>
+        <mesh filename="package://sprinter_description/meshes/lens_Yrot.stl" scale="0.001 0.001 0.001"/>
       </geometry>
       <material name="silver"/>
@@ -261,9 +261,9 @@
       <origin xyz="-0.144866 -0.270552 -0.528953" rpy="0 0 0"/>
       <geometry>
-        <mesh filename="package://sprinter_description/meshes/lens_Yrot_frame.stl" scale="0.001 0.001 0.001"/>
-      </geometry>
-    </collision>
-  </link>
-  <link name="lens_Xrot_frame">
+        <mesh filename="package://sprinter_description/meshes/lens_Yrot.stl" scale="0.001 0.001 0.001"/>
+      </geometry>
+    </collision>
+  </link>
+  <link name="lens_Xrot">
     <inertial>
       <origin xyz="-0.2533217422271652 7.584721687383723e-06 0.0013476837862036462" rpy="0 0 0"/>
@@ -274,5 +274,5 @@
       <origin xyz="-0.392366 8.1e-05 -0.552581" rpy="0 0 0"/>
       <geometry>
-        <mesh filename="package://sprinter_description/meshes/lens_Xrot_frame.stl" scale="0.001 0.001 0.001"/>
+        <mesh filename="package://sprinter_description/meshes/lens_Xrot.stl" scale="0.001 0.001 0.001"/>
       </geometry>
       <material name="silver"/>
@@ -281,5 +281,5 @@
       <origin xyz="-0.392366 8.1e-05 -0.552581" rpy="0 0 0"/>
       <geometry>
-        <mesh filename="package://sprinter_description/meshes/lens_Xrot_frame.stl" scale="0.001 0.001 0.001"/>
+        <mesh filename="package://sprinter_description/meshes/lens_Xrot.stl" scale="0.001 0.001 0.001"/>
       </geometry>
     </collision>
@@ -368,5 +368,5 @@
     <origin xyz="0.1445 -0.020515 0.143" rpy="0 0 0"/>
     <parent link="main_frame"/>
-    <child link="lens_Ylin_frame"/>
+    <child link="lens_Ylin"/>
     <axis xyz="0.0 1.0 0.0"/>
     <limit upper="0.15" lower="-0.12" effort="100" velocity="100"/>
@@ -374,6 +374,6 @@
   <joint name="Lens_X_axis_trans" type="prismatic">
     <origin xyz="-0.3947 0.020515 0.04114" rpy="0 0 0"/>
-    <parent link="lens_Ylin_frame"/>
-    <child link="lens_Xlin_frame"/>
+    <parent link="lens_Ylin"/>
+    <child link="lens_Xlin"/>
     <axis xyz="1.0 -0.0 0.0"/>
     <limit upper="0.65" lower="0.0" effort="100" velocity="100"/>
@@ -381,6 +381,6 @@
   <joint name="Lens_Y_axis_rot" type="revolute">
     <origin xyz="0.395066 0.270552 0.034813" rpy="0 0 0"/>
-    <parent link="lens_Xlin_frame"/>
-    <child link="lens_Yrot_frame"/>
+    <parent link="lens_Xlin"/>
+    <child link="lens_Yrot"/>
     <axis xyz="0.0 0.999999 0.001376"/>
     <limit upper="0.698132" lower="-0.698132" effort="100" velocity="100"/>
@@ -388,6 +388,6 @@
   <joint name="Lens_X_axis_rot" type="revolute">
     <origin xyz="0.2475 -0.270633 0.023628" rpy="0 0 0"/>
-    <parent link="lens_Yrot_frame"/>
-    <child link="lens_Xrot_frame"/>
+    <parent link="lens_Yrot"/>
+    <child link="lens_Xrot"/>
     <axis xyz="1.0 -0.0 0.0"/>
     <limit upper="1.2" lower="-1.2" effort="100" velocity="100"/>
@@ -396,5 +396,5 @@
   <joint name="lens_frame_middle_joint" type="fixed">
     <origin xyz="-0.2535  0.0 0.0" rpy="0 0 0"/>
-    <parent link="lens_Xrot_frame"/>
+    <parent link="lens_Xrot"/>
     <child link="lens_frame_middle"/>
   </joint>

File: ROS_ws/src/sprinter_robot_model/config/gazebo_sPrinter.urdf (robot description, URDF)
Before this commit: robot sPrinter, 17 links, 16 joints
Links:
- removed link lens_Xlin_frame
- removed link lens_Xrot_frame
- removed link lens_Ylin_frame
- removed link lens_Yrot_frame
- added link lens_Xlin, mass 1.8074023885886255; collision mesh filename=package://sprinter_description/meshes/lens_Xlin.stl scale=0.001 0.001 0.001; visual mesh filename=package://sprinter_description/meshes/lens_Xlin.stl scale=0.001 0.001 0.001
- added link lens_Xrot, mass 6.552542872975625; collision mesh filename=package://sprinter_description/meshes/lens_Xrot.stl scale=0.001 0.001 0.001; visual mesh filename=package://sprinter_description/meshes/lens_Xrot.stl scale=0.001 0.001 0.001
- added link lens_Ylin, mass 8.115658394698128; collision mesh filename=package://sprinter_description/meshes/lens_Ylin.stl scale=0.001 0.001 0.001; visual mesh filename=package://sprinter_description/meshes/lens_Ylin.stl scale=0.001 0.001 0.001
- added link lens_Yrot, mass 1.6400641565943115; collision mesh filename=package://sprinter_description/meshes/lens_Yrot.stl scale=0.001 0.001 0.001; visual mesh filename=package://sprinter_description/meshes/lens_Yrot.stl scale=0.001 0.001 0.001
Joints:
- joint Lens_X_axis_rot: child lens_Xrot_frame -> lens_Xrot; parent lens_Yrot_frame -> lens_Yrot
- joint Lens_X_axis_trans: child lens_Xlin_frame -> lens_Xlin; parent lens_Ylin_frame -> lens_Ylin
- joint Lens_Y_axis_rot: child lens_Yrot_frame -> lens_Yrot; parent lens_Xlin_frame -> lens_Xlin
- joint Lens_Y_axis_trans: child lens_Ylin_frame -> lens_Ylin
- joint lens_frame_middle_joint: parent lens_Xrot_frame -> lens_Xrot

Commit message: lensframe_middle -> lens_middle

File: ROS_ws/src/sprinter_description/urdf/sPrinter.urdf (robot description, URDF)
Before this commit: robot sPrinter, 17 links, 16 joints
Links:
- removed link lens_frame_middle
- added link lens_middle, mass 0.0
Joints:
- removed joint lens_frame_middle_joint
- added joint lens_middle_joint: type fixed, parent lens_Xrot, child lens_middle, origin xyz=-0.2535  0.0 0.0 rpy=0 0 0
- joint lens_focal_work_frame_joint: parent lens_frame_middle -> lens_middle

File: ROS_ws/src/sprinter_description/urdf/sPrinter.xacro (robot description, xacro)
@@ -286,5 +286,5 @@
   </link>
   <!--  frame in the middle of the lens-->
-  <link name="lens_frame_middle">
+  <link name="lens_middle">
     <inertial>
       <origin xyz="0.0 0.0 0.0" rpy="0 0 0"/>
@@ -394,8 +394,8 @@
   </joint>
   <!--middle frame joint-->
-  <joint name="lens_frame_middle_joint" type="fixed">
+  <joint name="lens_middle_joint" type="fixed">
     <origin xyz="-0.2535  0.0 0.0" rpy="0 0 0"/>
     <parent link="lens_Xrot"/>
-    <child link="lens_frame_middle"/>
+    <child link="lens_middle"/>
   </joint>
   <!--focal work frame joint-->
@@ -403,5 +403,5 @@
     <origin rpy="0 0 0" xyz="0.0 0.0 -0.55" />
             <!-- z: ohniskova vzdialenost -->
-    <parent link="lens_frame_middle"/>
+    <parent link="lens_middle"/>
     <child link="lens_focal_work_frame"/>
   </joint>

File: ROS_ws/src/sprinter_robot_model/config/gazebo_sPrinter.urdf (robot description, URDF)
Before this commit: robot sPrinter, 17 links, 16 joints
Links:
- removed link lens_frame_middle
- added link lens_middle, mass 0.0
Joints:
- removed joint lens_frame_middle_joint
- added joint lens_middle_joint: type fixed, parent lens_Xrot, child lens_middle, origin xyz=-0.2535  0.0 0.0 rpy=0 0 0
- joint lens_focal_work_frame_joint: parent lens_frame_middle -> lens_middle
