Commit message: added "_link" to links

File: ROS_ws/src/sprinter_description/urdf/sPrinter.urdf (robot description, URDF)
Before this commit: robot sPrinter, 17 links, 16 joints
Links:
- removed link boggie_left
- removed link boggie_right
- removed link lens_Xlin
- removed link lens_Xrot
- removed link lens_Ylin
- removed link lens_Yrot
- removed link lens_middle
- removed link main_frame
- removed link wheel_left_front
- removed link wheel_left_middle
- removed link wheel_left_rear
- removed link wheel_right_front
- removed link wheel_right_middle
- removed link wheel_right_rear
- added link boggie_left_link, mass 9.26099437267114; collision mesh filename=package://sprinter_description/meshes/boggie_left.stl scale=0.001 0.001 0.001; visual mesh filename=package://sprinter_description/meshes/boggie_left.stl scale=0.001 0.001 0.001
- added link boggie_right_link, mass 9.260994382343632; collision mesh filename=package://sprinter_description/meshes/boggie_right.stl scale=0.001 0.001 0.001; visual mesh filename=package://sprinter_description/meshes/boggie_right.stl scale=0.001 0.001 0.001
- added link lens_Xlin_link, mass 1.8074023885886255; collision mesh filename=package://sprinter_description/meshes/lens_Xlin.stl scale=0.001 0.001 0.001; visual mesh filename=package://sprinter_description/meshes/lens_Xlin.stl scale=0.001 0.001 0.001
- added link lens_Xrot_link, mass 6.552542872975625; collision mesh filename=package://sprinter_description/meshes/lens_Xrot.stl scale=0.001 0.001 0.001; visual mesh filename=package://sprinter_description/meshes/lens_Xrot.stl scale=0.001 0.001 0.001
- added link lens_Ylin_link, mass 8.115658394698128; collision mesh filename=package://sprinter_description/meshes/lens_Ylin.stl scale=0.001 0.001 0.001; visual mesh filename=package://sprinter_description/meshes/lens_Ylin.stl scale=0.001 0.001 0.001
- added link lens_Yrot_link, mass 1.6400641565943115; collision mesh filename=package://sprinter_description/meshes/lens_Yrot.stl scale=0.001 0.001 0.001; visual mesh filename=package://sprinter_description/meshes/lens_Yrot.stl scale=0.001 0.001 0.001
- added link lens_middle_link, mass 0.0
- added link main_frame_link, mass 37.61630562888167; collision mesh filename=package://sprinter_description/meshes/main_frame.stl scale=0.001 0.001 0.001; visual mesh filename=package://sprinter_description/meshes/main_frame.stl scale=0.001 0.001 0.001
- added link wheel_left_front_link, mass 16.78468038884107; collision mesh filename=package://sprinter_description/meshes/wheel_left_front.stl scale=0.001 0.001 0.001; visual mesh filename=package://sprinter_description/meshes/wheel_left_front.stl scale=0.001 0.001 0.001
- added link wheel_left_middle_link, mass 16.784680388841238; collision mesh filename=package://sprinter_description/meshes/wheel_left_middle.stl scale=0.001 0.001 0.001; visual mesh filename=package://sprinter_description/meshes/wheel_left_middle.stl scale=0.001 0.001 0.001
- added link wheel_left_rear_link, mass 16.7846803888409; collision mesh filename=package://sprinter_description/meshes/wheel_left_rear.stl scale=0.001 0.001 0.001; visual mesh filename=package://sprinter_description/meshes/wheel_left_rear.stl scale=0.001 0.001 0.001
- added link wheel_right_front_link, mass 16.784680388840883; collision mesh filename=package://sprinter_description/meshes/wheel_right_front.stl scale=0.001 0.001 0.001; visual mesh filename=package://sprinter_description/meshes/wheel_right_front.stl scale=0.001 0.001 0.001
- added link wheel_right_middle_link, mass 16.784680388841224; collision mesh filename=package://sprinter_description/meshes/wheel_right_middle.stl scale=0.001 0.001 0.001; visual mesh filename=package://sprinter_description/meshes/wheel_right_middle.stl scale=0.001 0.001 0.001
- added link wheel_right_rear_link, mass 16.78468038884136; collision mesh filename=package://sprinter_description/meshes/wheel_right_rear.stl scale=0.001 0.001 0.001; visual mesh filename=package://sprinter_description/meshes/wheel_right_rear.stl scale=0.001 0.001 0.001
Joints:
- joint Boggie_left: child boggie_left -> boggie_left_link
- joint Boggie_right: child boggie_right -> boggie_right_link
- joint Lens_X_axis_rot: child lens_Xrot -> lens_Xrot_link; parent lens_Yrot -> lens_Yrot_link
- joint Lens_X_axis_trans: child lens_Xlin -> lens_Xlin_link; parent lens_Ylin -> lens_Ylin_link
- joint Lens_Y_axis_rot: child lens_Yrot -> lens_Yrot_link; parent lens_Xlin -> lens_Xlin_link
- joint Lens_Y_axis_trans: child lens_Ylin -> lens_Ylin_link; parent main_frame -> main_frame_link
- joint MainFrame_pitch: child main_frame -> main_frame_link
- joint Wheel_left_front: child wheel_left_front -> wheel_left_front_link
- joint Wheel_left_middle: child wheel_left_middle -> wheel_left_middle_link; parent boggie_left -> boggie_left_link
- joint Wheel_left_rear: child wheel_left_rear -> wheel_left_rear_link; parent boggie_left -> boggie_left_link
- joint Wheel_right_front: child wheel_right_front -> wheel_right_front_link
- joint Wheel_right_middle: child wheel_right_middle -> wheel_right_middle_link; parent boggie_right -> boggie_right_link
- joint Wheel_right_rear: child wheel_right_rear -> wheel_right_rear_link; parent boggie_right -> boggie_right_link
- joint lens_focal_work_frame_joint: parent lens_middle -> lens_middle_link
- joint lens_middle_joint: child lens_middle -> lens_middle_link; parent lens_Xrot -> lens_Xrot_link

File: ROS_ws/src/sprinter_description/urdf/sPrinter.xacro (robot description, xacro)
@@ -25,5 +25,5 @@
     </collision>
   </link>
-  <link name="boggie_right">
+  <link name="boggie_right_link">
     <inertial>
       <origin xyz="0.04608835670723324 -0.05868381694977415 -0.08782934708885383" rpy="0 0 0"/>
@@ -45,5 +45,5 @@
     </collision>
   </link>
-  <link name="boggie_left">
+  <link name="boggie_left_link">
     <inertial>
       <origin xyz="0.04608852267144553 0.05868381722034843 -0.0878295588540255" rpy="0 0 0"/>
@@ -65,5 +65,5 @@
     </collision>
   </link>
-  <link name="wheel_right_front">
+  <link name="wheel_right_front_link">
     <inertial>
       <origin xyz="-2.2157215140428121e-07 0.049038331285879255 -5.319570878098423e-07" rpy="0 0 0"/>
@@ -85,5 +85,5 @@
     </collision>
   </link>
-  <link name="wheel_right_middle">
+  <link name="wheel_right_middle_link">
     <inertial>
       <origin xyz="-2.441464656044445e-07 0.049038331285878034 -1.2471173249650747e-07" rpy="0 0 0"/>
@@ -105,5 +105,5 @@
     </collision>
   </link>
-  <link name="wheel_right_rear">
+  <link name="wheel_right_rear_link">
     <inertial>
       <origin xyz="-2.4414526850202733e-07 0.04903833128586854 4.1045225383784523e-07" rpy="0 0 0"/>
@@ -125,5 +125,5 @@
     </collision>
   </link>
-  <link name="wheel_left_front">
+  <link name="wheel_left_front_link">
     <inertial>
       <origin xyz="-1.7782965933133e-08 -0.04903833128669849 -7.65968576066367e-08" rpy="0 0 0"/>
@@ -145,5 +145,5 @@
     </collision>
   </link>
-  <link name="wheel_left_middle">
+  <link name="wheel_left_middle_link">
     <inertial>
       <origin xyz="1.038819750736053e-06 -0.049038331286717474 0.00010982563519425226" rpy="0 0 0"/>
@@ -165,5 +165,5 @@
     </collision>
   </link>
-  <link name="wheel_left_rear">
+  <link name="wheel_left_rear_link">
     <inertial>
       <origin xyz="1.0388197915767172e-06 -0.04903833128671531 0.00010972160107960982" rpy="0 0 0"/>
@@ -185,5 +185,5 @@
     </collision>
   </link>
-  <link name="main_frame">
+  <link name="main_frame_link">
     <inertial>
       <origin xyz="-0.08748571926603223 0.002858790568392067 -0.009190179413522459" rpy="0 0 0"/>
@@ -205,5 +205,5 @@
     </collision>
   </link>
-  <link name="lens_Ylin">
+  <link name="lens_Ylin_link">
     <inertial>
       <origin xyz="-0.19050492237401995 0.01911574728140262 0.050354275554037764" rpy="0 0 0"/>
@@ -225,5 +225,5 @@
     </collision>
   </link>
-  <link name="lens_Xlin">
+  <link name="lens_Xlin_link">
     <inertial>
       <origin xyz="0.23595566779369742 0.13671241587093597 0.03333844333172431" rpy="0 0 0"/>
@@ -245,5 +245,5 @@
     </collision>
   </link>
-  <link name="lens_Yrot">
+  <link name="lens_Yrot_link">
     <inertial>
       <origin xyz="0.15610000473558938 -0.28034931010215036 0.01290803779832872" rpy="0 0 0"/>
@@ -265,5 +265,5 @@
     </collision>
   </link>
-  <link name="lens_Xrot">
+  <link name="lens_Xrot_link">
     <inertial>
       <origin xyz="-0.2533217422271652 7.584721687383723e-06 0.0013476837862036462" rpy="0 0 0"/>
@@ -286,5 +286,5 @@
   </link>
   <!--  frame in the middle of the lens-->
-  <link name="lens_middle">
+  <link name="lens_middle_link">
     <inertial>
       <origin xyz="0.0 0.0 0.0" rpy="0 0 0"/>
@@ -311,5 +311,5 @@
     <origin xyz="-0.26 -0.22975 0.21" rpy="0 0 0"/>
     <parent link="base_link"/>
-    <child link="boggie_right"/>
+    <child link="boggie_right_link"/>
     <axis xyz="-0.0 1.0 0.0"/>
     <limit upper="0.523599" lower="-0.523599" effort="100" velocity="100"/>
@@ -318,5 +318,5 @@
     <origin xyz="-0.26 0.22975 0.21" rpy="0 0 0"/>
     <parent link="base_link"/>
-    <child link="boggie_left"/>
+    <child link="boggie_left_link"/>
     <axis xyz="0.0 1.0 0.0"/>
     <limit upper="0.523599" lower="-0.523599" effort="100" velocity="100"/>
@@ -325,17 +325,17 @@
     <origin xyz="0.42 -0.38275 0.09" rpy="0 0 0"/>
     <parent link="base_link"/>
-    <child link="wheel_right_front"/>
+    <child link="wheel_right_front_link"/>
     <axis xyz="0.0 1.0 0.0"/>
   </joint>
   <joint name="Wheel_right_middle" type="continuous">
     <origin xyz="0.26 -0.174 -0.12" rpy="0 0 0"/>
-    <parent link="boggie_right"/>
-    <child link="wheel_right_middle"/>
+    <parent link="boggie_right_link"/>
+    <child link="wheel_right_middle_link"/>
     <axis xyz="0.0 1.0 0.0"/>
   </joint>
   <joint name="Wheel_right_rear" type="continuous">
     <origin xyz="-0.16 -0.174 -0.12" rpy="0 0 0"/>
-    <parent link="boggie_right"/>
-    <child link="wheel_right_rear"/>
+    <parent link="boggie_right_link"/>
+    <child link="wheel_right_rear_link"/>
     <axis xyz="0.0 1.0 0.0"/>
   </joint>
@@ -343,17 +343,17 @@
     <origin xyz="0.42 0.38275 0.09" rpy="0 0 0"/>
     <parent link="base_link"/>
-    <child link="wheel_left_front"/>
+    <child link="wheel_left_front_link"/>
     <axis xyz="0.0 1.0 0.0"/>
   </joint>
   <joint name="Wheel_left_middle" type="continuous">
     <origin xyz="0.26 0.174 -0.12" rpy="0 0 0"/>
-    <parent link="boggie_left"/>
-    <child link="wheel_left_middle"/>
+    <parent link="boggie_left_link"/>
+    <child link="wheel_left_middle_link"/>
     <axis xyz="0.0 1.0 0.0"/>
   </joint>
   <joint name="Wheel_left_rear" type="continuous">
     <origin xyz="-0.16 0.174 -0.12" rpy="0 0 0"/>
-    <parent link="boggie_left"/>
-    <child link="wheel_left_rear"/>
+    <parent link="boggie_left_link"/>
+    <child link="wheel_left_rear_link"/>
     <axis xyz="0.0 1.0 0.0"/>
   </joint>
@@ -361,5 +361,5 @@
     <origin xyz="0.0 0.0 0.31" rpy="0 0 0"/>
     <parent link="base_link"/>
-    <child link="main_frame"/>
+    <child link="main_frame_link"/>
     <axis xyz="-0.0 1.0 0.0"/>
     <limit upper="0.523599" lower="-0.523599" effort="100" velocity="100"/>
@@ -367,6 +367,6 @@
   <joint name="Lens_Y_axis_trans" type="prismatic">
     <origin xyz="0.1445 -0.020515 0.143" rpy="0 0 0"/>
-    <parent link="main_frame"/>
-    <child link="lens_Ylin"/>
+    <parent link="main_frame_link"/>
+    <child link="lens_Ylin_link"/>
     <axis xyz="0.0 1.0 0.0"/>
     <limit upper="0.15" lower="-0.12" effort="100" velocity="100"/>
@@ -374,6 +374,6 @@
   <joint name="Lens_X_axis_trans" type="prismatic">
     <origin xyz="-0.3947 0.020515 0.04114" rpy="0 0 0"/>
-    <parent link="lens_Ylin"/>
-    <child link="lens_Xlin"/>
+    <parent link="lens_Ylin_link"/>
+    <child link="lens_Xlin_link"/>
     <axis xyz="1.0 -0.0 0.0"/>
     <limit upper="0.65" lower="0.0" effort="100" velocity="100"/>
@@ -381,6 +381,6 @@
   <joint name="Lens_Y_axis_rot" type="revolute">
     <origin xyz="0.395066 0.270552 0.034813" rpy="0 0 0"/>
-    <parent link="lens_Xlin"/>
-    <child link="lens_Yrot"/>
+    <parent link="lens_Xlin_link"/>
+    <child link="lens_Yrot_link"/>
     <axis xyz="0.0 0.999999 0.001376"/>
     <limit upper="0.698132" lower="-0.698132" effort="100" velocity="100"/>
@@ -388,6 +388,6 @@
   <joint name="Lens_X_axis_rot" type="revolute">
     <origin xyz="0.2475 -0.270633 0.023628" rpy="0 0 0"/>
-    <parent link="lens_Yrot"/>
-    <child link="lens_Xrot"/>
+    <parent link="lens_Yrot_link"/>
+    <child link="lens_Xrot_link"/>
     <axis xyz="1.0 -0.0 0.0"/>
     <limit upper="1.2" lower="-1.2" effort="100" velocity="100"/>
@@ -396,6 +396,6 @@
   <joint name="lens_middle_joint" type="fixed">
     <origin xyz="-0.2535  0.0 0.0" rpy="0 0 0"/>
-    <parent link="lens_Xrot"/>
-    <child link="lens_middle"/>
+    <parent link="lens_Xrot_link"/>
+    <child link="lens_middle_link"/>
   </joint>
   <!--focal work frame joint-->
@@ -403,5 +403,5 @@
     <origin rpy="0 0 0" xyz="0.0 0.0 -0.55" />
             <!-- z: ohniskova vzdialenost -->
-    <parent link="lens_middle"/>
+    <parent link="lens_middle_link"/>
     <child link="lens_focal_work_frame"/>
   </joint>

File: ROS_ws/src/sprinter_robot_model/config/gazebo_sPrinter.urdf (robot description, URDF)
Before this commit: robot sPrinter, 17 links, 16 joints
Links:
- removed link boggie_left
- removed link boggie_right
- removed link lens_Xlin
- removed link lens_Xrot
- removed link lens_Ylin
- removed link lens_Yrot
- removed link lens_middle
- removed link main_frame
- removed link wheel_left_front
- removed link wheel_left_middle
- removed link wheel_left_rear
- removed link wheel_right_front
- removed link wheel_right_middle
- removed link wheel_right_rear
- added link boggie_left_link, mass 9.26099437267114; collision mesh filename=package://sprinter_description/meshes/boggie_left.stl scale=0.001 0.001 0.001; visual mesh filename=package://sprinter_description/meshes/boggie_left.stl scale=0.001 0.001 0.001
- added link boggie_right_link, mass 9.260994382343632; collision mesh filename=package://sprinter_description/meshes/boggie_right.stl scale=0.001 0.001 0.001; visual mesh filename=package://sprinter_description/meshes/boggie_right.stl scale=0.001 0.001 0.001
- added link lens_Xlin_link, mass 1.8074023885886255; collision mesh filename=package://sprinter_description/meshes/lens_Xlin.stl scale=0.001 0.001 0.001; visual mesh filename=package://sprinter_description/meshes/lens_Xlin.stl scale=0.001 0.001 0.001
- added link lens_Xrot_link, mass 6.552542872975625; collision mesh filename=package://sprinter_description/meshes/lens_Xrot.stl scale=0.001 0.001 0.001; visual mesh filename=package://sprinter_description/meshes/lens_Xrot.stl scale=0.001 0.001 0.001
- added link lens_Ylin_link, mass 8.115658394698128; collision mesh filename=package://sprinter_description/meshes/lens_Ylin.stl scale=0.001 0.001 0.001; visual mesh filename=package://sprinter_description/meshes/lens_Ylin.stl scale=0.001 0.001 0.001
- added link lens_Yrot_link, mass 1.6400641565943115; collision mesh filename=package://sprinter_description/meshes/lens_Yrot.stl scale=0.001 0.001 0.001; visual mesh filename=package://sprinter_description/meshes/lens_Yrot.stl scale=0.001 0.001 0.001
- added link lens_middle_link, mass 0.0
- added link main_frame_link, mass 37.61630562888167; collision mesh filename=package://sprinter_description/meshes/main_frame.stl scale=0.001 0.001 0.001; visual mesh filename=package://sprinter_description/meshes/main_frame.stl scale=0.001 0.001 0.001
- added link wheel_left_front_link, mass 16.78468038884107; collision mesh filename=package://sprinter_description/meshes/wheel_left_front.stl scale=0.001 0.001 0.001; visual mesh filename=package://sprinter_description/meshes/wheel_left_front.stl scale=0.001 0.001 0.001
- added link wheel_left_middle_link, mass 16.784680388841238; collision mesh filename=package://sprinter_description/meshes/wheel_left_middle.stl scale=0.001 0.001 0.001; visual mesh filename=package://sprinter_description/meshes/wheel_left_middle.stl scale=0.001 0.001 0.001
- added link wheel_left_rear_link, mass 16.7846803888409; collision mesh filename=package://sprinter_description/meshes/wheel_left_rear.stl scale=0.001 0.001 0.001; visual mesh filename=package://sprinter_description/meshes/wheel_left_rear.stl scale=0.001 0.001 0.001
- added link wheel_right_front_link, mass 16.784680388840883; collision mesh filename=package://sprinter_description/meshes/wheel_right_front.stl scale=0.001 0.001 0.001; visual mesh filename=package://sprinter_description/meshes/wheel_right_front.stl scale=0.001 0.001 0.001
- added link wheel_right_middle_link, mass 16.784680388841224; collision mesh filename=package://sprinter_description/meshes/wheel_right_middle.stl scale=0.001 0.001 0.001; visual mesh filename=package://sprinter_description/meshes/wheel_right_middle.stl scale=0.001 0.001 0.001
- added link wheel_right_rear_link, mass 16.78468038884136; collision mesh filename=package://sprinter_description/meshes/wheel_right_rear.stl scale=0.001 0.001 0.001; visual mesh filename=package://sprinter_description/meshes/wheel_right_rear.stl scale=0.001 0.001 0.001
Joints:
- joint Boggie_left: child boggie_left -> boggie_left_link
- joint Boggie_right: child boggie_right -> boggie_right_link
- joint Lens_X_axis_rot: child lens_Xrot -> lens_Xrot_link; parent lens_Yrot -> lens_Yrot_link
- joint Lens_X_axis_trans: child lens_Xlin -> lens_Xlin_link; parent lens_Ylin -> lens_Ylin_link
- joint Lens_Y_axis_rot: child lens_Yrot -> lens_Yrot_link; parent lens_Xlin -> lens_Xlin_link
- joint Lens_Y_axis_trans: child lens_Ylin -> lens_Ylin_link; parent main_frame -> main_frame_link
- joint MainFrame_pitch: child main_frame -> main_frame_link
- joint Wheel_left_front: child wheel_left_front -> wheel_left_front_link
- joint Wheel_left_middle: child wheel_left_middle -> wheel_left_middle_link; parent boggie_left -> boggie_left_link
- joint Wheel_left_rear: child wheel_left_rear -> wheel_left_rear_link; parent boggie_left -> boggie_left_link
- joint Wheel_right_front: child wheel_right_front -> wheel_right_front_link
- joint Wheel_right_middle: child wheel_right_middle -> wheel_right_middle_link; parent boggie_right -> boggie_right_link
- joint Wheel_right_rear: child wheel_right_rear -> wheel_right_rear_link; parent boggie_right -> boggie_right_link
- joint lens_focal_work_frame_joint: parent lens_middle -> lens_middle_link
- joint lens_middle_joint: child lens_middle -> lens_middle_link; parent lens_Xrot -> lens_Xrot_link

Commit message: renamed work and static lens frames

File: ROS_ws/src/sprinter_description/urdf/sPrinter.urdf (robot description, URDF)
Before this commit: robot sPrinter, 17 links, 16 joints
Links:
- removed link lens_focal_static_frame
- removed link lens_focal_work_frame
- added link lens_focal, mass 0.0
- added link ref_print_space, mass 0.0
Joints:
- removed joint lens_focal_static_frame_joint
- removed joint lens_focal_work_frame_joint
- added joint lens_focal_joint: type fixed, parent lens_middle_link, child lens_focal, origin xyz=0.0 0.0 -0.55 rpy=0 0 0
- added joint ref_print_space_joint: type fixed, parent base_link, child ref_print_space, origin xyz=0.753764 0.0 -0.0 rpy=0 0 0

File: ROS_ws/src/sprinter_description/urdf/sPrinter.xacro (robot description, xacro)
@@ -293,5 +293,5 @@
     </inertial>
   </link>
-  <link name="lens_focal_work_frame">
+  <link name="lens_focal">
     <inertial>
       <origin xyz="0.0 0.0 0.0" rpy="0 0 0"/>
@@ -300,5 +300,5 @@
     </inertial>
   </link>
-  <link name="lens_focal_static_frame">
+  <link name="ref_print_space">
     <inertial>
       <origin xyz="0.0 0.0 0.0" rpy="0 0 0"/>
@@ -400,17 +400,17 @@
   </joint>
   <!--focal work frame joint-->
-  <joint name="lens_focal_work_frame_joint" type="fixed">
+  <joint name="lens_focal_joint" type="fixed">
     <origin rpy="0 0 0" xyz="0.0 0.0 -0.55" />
             <!-- z: ohniskova vzdialenost -->
     <parent link="lens_middle_link"/>
-    <child link="lens_focal_work_frame"/>
+    <child link="lens_focal"/>
   </joint>
   <!--focal static frame joint-->
-  <joint name="lens_focal_static_frame_joint" type="fixed">
+  <joint name="ref_print_space_joint" type="fixed">
     <origin rpy="0 0 0" xyz="0.753764 0.0 -0.0" />
             <!-- z: -55cm - ohniskova vzdialenost = 0cm nad rovinou zeme-->
-            <!-- x: 0.753764 je pri 0.615m vysunuti sosovky v x (HOME) ... pod lens_midle frame-->
-    <parent link="base_link"/>
-    <child link="lens_focal_static_frame"/>
+            <!-- x: 0.753764 je pri 0.615m vysunuti sosovky v x (HOME) ... pod lens_middle frame-->
+    <parent link="base_link"/>
+    <child link="ref_print_space"/>
   </joint>
 </robot>

File: ROS_ws/src/sprinter_robot_model/config/gazebo_sPrinter.urdf (robot description, URDF)
Before this commit: robot sPrinter, 17 links, 16 joints
Links:
- removed link lens_focal_static_frame
- removed link lens_focal_work_frame
- added link lens_focal, mass 0.0
- added link ref_print_space, mass 0.0
Joints:
- removed joint lens_focal_static_frame_joint
- removed joint lens_focal_work_frame_joint
- added joint lens_focal_joint: type fixed, parent lens_middle_link, child lens_focal, origin xyz=0.0 0.0 -0.55 rpy=0 0 0
- added joint ref_print_space_joint: type fixed, parent base_link, child ref_print_space, origin xyz=0.753764 0.0 -0.0 rpy=0 0 0
